Commit message: rizon4: wrap bare origin/mass/inertia triples in <inertial> (flexiv xacro defect; values cross-checked vs mujoco_menagerie) — zero-inertia skips self-heal

File: robot_assets/rizon4.urdf (robot description, URDF)
Before this commit: robot Rizon4, 10 links, 9 joints
Links:
- link base_link: mass None -> 3.8
- link link1: mass None -> 3.6
- link link2: mass None -> 2.7
- link link3: mass None -> 2.4
- link link4: mass None -> 2.4
- link link5: mass None -> 2.3
- link link6: mass None -> 2.2
- link link7: mass None -> 0.8
